Commit message: added D435

File: urdf/lb_description.urdf.xacro (robot description, xacro)
@@ -1,6 +1,12 @@
 <?xml version="1.0"?>
-<robot xmlns:xacro="http://www.ros.org/wiki/xacro" name="littlebot">
-  <link name="base_link">
-  </link>
+<robot name="littlebot" xmlns:xacro="http://www.ros.org/wiki/xacro">
+  <xacro:arg name="use_nominal_extrinsics" default="true"/>
+  <xacro:arg name="add_plug" default="false" />
+  <xacro:arg name="use_mesh" default="true" />
+  <xacro:include filename="$(find realsense2_description)/urdf/_d435.urdf.xacro" />
+  <link name="base_link"/>
+  <xacro:sensor_d435 parent="chassis_link" use_nominal_extrinsics="$(arg use_nominal_extrinsics)" add_plug="$(arg add_plug)" use_mesh="$(arg use_mesh)">
+    <origin xyz="-0.13 0.105 0.005" rpy="0 0 1.57079"/>
+  </xacro:sensor_d435>
   <link name="wheel1_link">
     <inertial>
@@ -196,7 +202,4 @@
     <axis xyz="0 0 1" />
   </joint>
-  <!-- Import lb ros2_control description
-  <xacro:include filename="$(find lb_description)/ros2_control/lb_ros2_control.xacro" />
-  <xacro:lb_ros2_control name="littlebot" /> -->
   <ros2_control name="lb_base_controller" type="system">
     <hardware>
